Commit message: Added multicamera and fine-tuned config parameters

File: husky_fei_description/urdf/husky_fei.urdf (robot description, URDF)
Before this commit: robot husky_fei, 10 links, 9 joints
Links:
- added link baro_link, mass 0.10; visual box size=0.01 0.02 0.02
- added link base_footprint_fei_cam_rail_part, mass 0.1; collision box size=0.02 0.02 0.3; visual mesh filename=package://husky_fei_description/meshes/tslot_300x20x20.dae
- added link base_footprint_fei_gps_rail_part, mass 0.1; collision box size=0.02 0.02 0.4; visual mesh filename=package://husky_fei_description/meshes/tslot_400x20x20.dae
- added link base_footprint_fei_hb_rail_part, mass 0.1; collision box size=0.001 0.001 0.001; visual mesh filename=package://husky_fei_description/meshes/tslot_400x20x20.dae
- added link base_footprint_fei_hf_rail_part, mass 0.1; collision box size=0.001 0.001 0.001; visual mesh filename=package://husky_fei_description/meshes/tslot_400x20x20.dae
- added link base_footprint_fei_lms100_l_rail_part, mass 0.1; collision box size=0.02 0.02 0.1; visual mesh filename=package://husky_fei_description/meshes/tslot_100x20x20.dae
- added link base_footprint_fei_lms100_r_rail_part, mass 0.1; collision box size=0.02 0.02 0.1; visual mesh filename=package://husky_fei_description/meshes/tslot_100x20x20.dae
- added link base_footprint_lms100_support_part, mass 0.1; collision box size=0.02 0.02 0.1; visual mesh filename=package://husky_fei_description/meshes/sensors/LMS100_suppo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
- added link gps_link, mass 0.10; collision box size=0.16 0.16 0.16; visual mesh filename=package://husky_fei_description/meshes/sensors/GPSAntenna.d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
- added link imu_link, mass 0.01; visual box size=0.025 0.025 0.01
- added link laser_link, mass 1.1; collision box size=0.120 0.102 0.165; visual mesh filename=package://husky_fei_description/meshes/sensors/LMS100.dae
- added link left_camera_frame; visual cylinder length=0.01 radius=0.01
- added link right_camera_frame; visual cylinder length=0.01 radius=0.01
- added link stereo_camera_link, mass 0.01; collision box size=0.05 0.1 0.05; visual box size=0.05 0.1 0.05
Joints:
- added joint baro_joint: type fixed, parent base_link, child baro_link, origin xyz=0.192 -0.05 0.19492492 rpy=0.0 0.0 0.0
- added joint base_footprint_fei_cam_rail_joint: type fixed, parent base_footprint, child base_footprint_fei_cam_rail_part, origin xyz=-0.15 0.0 0.54092492 rpy=0.0 0.0 0.0
- added joint base_footprint_fei_gps_rail_joint: type fixed, parent base_footprint, child base_footprint_fei_gps_rail_part, origin xyz=-0.15 0.18 0.58092492 rpy=1.57079632679 0.0 0.0
- added joint base_footprint_fei_hb_rail_joint: type fixed, parent base_footprint, child base_footprint_fei_hb_rail_part, origin xyz=-0.15 0.0 0.38092492 rpy=0.0 0.0 0.0
- added joint base_footprint_fei_hf_rail_joint: type fixed, parent base_footprint, child base_footprint_fei_hf_rail_part, origin xyz=0.21 0.0 0.38092492 rpy=0.0 0.0 0.0
- added joint base_footprint_fei_lms100_l_rail_joint: type fixed, parent base_footprint, child base_footprint_fei_lms100_l_rail_part, origin xyz=0.242 -0.035 0.42092492 rpy=0.0 0.0 0.0
- added joint base_footprint_fei_lms100_r_rail_joint: type fixed, parent base_footprint, child base_footprint_fei_lms100_r_rail_part, origin xyz=0.242 0.035 0.42092492 rpy=0.0 0.0 0.0
- added joint base_footprint_lms100_support_joint: type fixed, parent base_footprint, child base_footprint_lms100_support_part, origin xyz=0.314 0.0 0.47992492 rpy=0.0 0.0 0.0
- added joint gps_joint: type fixed, parent base_link, child gps_link, origin xyz=-0.151 0.182 0.61392492 rpy=0.0 0.0 3.14159265359
- added joint imu_joint: type fixed, parent base_link, child imu_link, origin xyz=0.192 0.0 0.19492492 rpy=0.0 -1.57079632679 0.0
- added joint laser_joint: type fixed, parent base_link, child laser_link, origin xyz=0.314 0.0 0.28492492 rpy=0.0 0.0 0
- added joint left_camera_joint: type fixed, parent stereo_camera_link, child left_camera_frame, origin xyz=0 0.031 0 rpy=0 0 0
- added joint right_camera_joint: type fixed, parent stereo_camera_link, child right_camera_frame, origin xyz=0 -0.031 0 rpy=0 0 0
- added joint stereo_camera_joint: type fixed, parent base_link, child stereo_camera_link, origin xyz=-0.15 0.0 0.54092492 rpy=0.0 0.0 0.0

File: husky_fei_description/urdf/husky_fei.urdf.xacro (robot description, xacro)
@@ -6,4 +6,5 @@
     <xacro:include filename="$(find husky_fei_description)/urdf/parts/parts.urdf.xacro" />
     <xacro:include filename="$(find husky_fei_description)/urdf/sensors/kinect.urdf.xacro" />
+    <xacro:include filename="$(find husky_fei_description)/urdf/sensors/multicamera.urdf.xacro" />
     <xacro:include filename="$(find husky_fei_description)/urdf/sensors/imu.urdf.xacro" />
     <xacro:include filename="$(find husky_fei_description)/urdf/sensors/gps.urdf.xacro" />
@@ -157,8 +158,21 @@
     </gazebo>
     <!-- FEI-modded 3D sensor -->
-    <sensor_kinect parent="base_link" cam_px="-0.12" cam_py="0.0" cam_pz="${0.207 + 0.245 + wheel_x_size/2 - base_z_origin_to_wheel_origin}" cam_or="0.0" cam_op="0.0" cam_oy="0.0" />
+<!--
+    <sensor_kinect name="camera" parent="base_link" cam_px="-0.12" cam_py="0.0" cam_pz="${0.207 + 0.245 + wheel_x_size/2 - base_z_origin_to_wheel_origin}" cam_or="0.0" cam_op="0.0" cam_oy="0.0" />
+-->
+    <!-- FEI-modded multicamera sensor -->
+    <sensor_multicamera name="stereo_camera" parent="base_link" baseline="0.062" colour="Red" cam_px="-0.15" cam_py="0.0" cam_pz="${0.151 + 0.245 + wheel_x_size/2 - base_z_origin_to_wheel_origin}" cam_or="0.0" cam_op="0.0" cam_oy="0.0" />
+    <gazebo reference="stereo_camera_link">
+        <material>Gazebo/Red</material>
+    </gazebo>
+    <gazebo reference="left_camera_frame">
+        <material>Gazebo/Black</material>
+    </gazebo>
+    <gazebo reference="right_camera_frame">
+        <material>Gazebo/Black</material>
+    </gazebo>
     <!-- FEI-modded IMU sensor -->
     <!--<sensor_imu name="imu" parent="base" colour="Blue" imu_px="0.192" imu_py="0.0" imu_pz="${0.05 + wheel_x_size/2 - base_z_origin_to_wheel_origin}" imu_or="0.0" imu_op="${M_PI/2.0}" imu_oy="0.0" imu_topic="imu_data" update_rate="100.0" stdev="1.7e-2" /> -->
-    <sensor_imu parent="base_link" name="imu" colour="Blue" imu_px="0.192" imu_py="0.0" imu_pz="${0.05 + wheel_x_size/2 - base_z_origin_to_wheel_origin}" imu_or="0.0" imu_op="${M_PI/2.0}" imu_oy="0.0" />
+    <sensor_imu parent="base_link" name="imu" colour="Blue" imu_px="0.192" imu_py="0.0" imu_pz="${0.05 + wheel_x_size/2 - base_z_origin_to_wheel_origin}" imu_or="0.0" imu_op="${-M_PI/2.0}" imu_oy="0.0" />
     <gazebo reference="imu_link">
         <material>Gazebo/Blue</material>

File: husky_fei_description/urdf/sensors/3dsensor_gazebo.urdf.xacro (robot description, xacro)
@@ -2,7 +2,7 @@
 <robot name="3dsensor_gazebo" xmlns:xacro="http://ros.org/wiki/xacro">
   <!-- Microsoft Kinect / ASUS Xtion PRO Live for simulation -->
-  <xacro:macro name="husky_fei_sim_3dsensor">
-    <gazebo reference="camera_link">
-      <sensor type="depth" name="camera">
+  <xacro:macro name="husky_fei_sim_3dsensor" params="name">
+    <gazebo reference="${name}_link">
+      <sensor type="depth" name="${name}">
         <always_on>true</always_on>
         <update_rate>30.0</update_rate>
@@ -19,8 +19,7 @@
           </clip>
         </camera>
-        <plugin name="kinect_camera_controller" filename="libgazebo_ros_openni_kinect.so">
-          <cameraName>camera</cameraName>
-          <alwaysOn>true</alwaysOn>
-          <updateRate>10.0</updateRate>
+        <plugin name="gazebo_ros_${name}_controller" filename="libgazebo_ros_openni_kinect.so">
+          <cameraName>${name}</cameraName>
+          <updateRate>30.0</updateRate>
           <imageTopicName>rgb/image_raw</imageTopicName>
           <depthImageTopicName>depth/image_raw</depthImageTopicName>
@@ -28,5 +27,5 @@
           <cameraInfoTopicName>rgb/camera_info</cameraInfoTopicName>
           <depthImageCameraInfoTopicName>depth/camera_info</depthImageCameraInfoTopicName>
-          <frameName>camera_depth_optical_frame</frameName>
+          <frameName>${name}_depth_optical_frame</frameName>
           <baseline>0.1</baseline>
           <distortion_k1>0.0</distortion_k1>

File: husky_fei_description/urdf/sensors/gps.urdf.xacro (robot description, xacro)
@@ -12,5 +12,5 @@
 	<origin xyz="0 0 0" rpy="0 0 0" />
 	<geometry>
-          <mesh filename="package://husky_fei_description/meshes/sensors/GPSAntenna.dae" />
+          <mesh filename="package://husky_fei_description/meshes/sensors/GPSAntennaScaledDown.dae" />
 	</geometry>
 	<material name="${colour}" />
@@ -19,5 +19,5 @@
         <origin rpy="0 0 0" xyz="0 0 0"/>
         <geometry>
-          <box size="${dimX} ${dimY} ${dimZ}"/>
+          <box size="${dimX * 0.6} ${dimY * 0.6} ${dimZ * 0.6}"/>
         </geometry>
       </collision>

File: husky_fei_description/urdf/sensors/imu.urdf.xacro (robot description, xacro)
@@ -6,5 +6,5 @@
       <inertial>
         <mass value="0.01"/>
-        <origin xyz="0 0 0"/>
+        <origin xyz="0 0 0" rpy="0 0 0" />
         <inertia ixx="0.000001" ixy="0" ixz="0" iyy="0.000001" iyz="0" izz="0.000001"/>
       </inertial>

File: husky_fei_description/urdf/sensors/kinect_camera.urdf.xacro (robot description, xacro)
@@ -11,36 +11,10 @@
   <xacro:include filename="$(find husky_fei_description)/urdf/sensors/3dsensor_gazebo.urdf.xacro"/>
   <xacro:macro name="sensor_kinect" params="name parent cam_px cam_py cam_pz cam_or cam_op cam_oy">
-    <joint name="${name}_joint" type="fixed">
-      <origin xyz="${cam_px - 0.031} ${cam_py} ${cam_pz - 0.016}" rpy="${cam_or} ${cam_op} ${cam_oy}"/>
+    <joint name="camera_rgb_joint" type="fixed">
+      <origin xyz="${cam_px} ${cam_py} ${cam_pz}" rpy="${cam_or} ${cam_op} ${cam_oy}"/>
       <parent link="${parent}"/>
-      <child link="${name}_link" />
+      <child link="camera_rgb_frame" />
     </joint>
-    <link name="${name}_link">
-      <inertial>
-        <mass value="0.001" />
-        <origin xyz="0 0 0" />
-        <inertia ixx="0.0001" ixy="0.0" ixz="0.0"
-                 iyy="0.0001" iyz="0.0"
-                 izz="0.0001" />
-      </inertial>
-      <visual>
-        <origin xyz="0 0 0" rpy="0 0 ${M_PI/2}"/>
-          <geometry>
-            <mesh filename="package://husky_fei_description/meshes/sensors/kinect.dae"/>
-          </geometry>
-      </visual>
-      <collision>
-        <origin xyz="0.0 0.0 0.0" rpy="0 0 0"/>
-        <geometry>
-          <box size="0.07271 0.27794 0.073"/>
-        </geometry>
-      </collision>
-    </link>
-    <joint name="${name}_rgb_joint" type="fixed">
-      <origin xyz="0.031 -0.0127 0.016" rpy="0 0 0"/>
-      <parent link="${name}_link"/>
-      <child link="${name}_rgb_frame"/>
-    </joint>
-    <link name="${name}_rgb_frame">
+    <link name="camera_rgb_frame">
       <inertial>
         <mass value="0.001" />
@@ -51,10 +25,10 @@
       </inertial>
     </link>
-    <joint name="${name}_rgb_optical_joint" type="fixed">
+    <joint name="camera_rgb_optical_joint" type="fixed">
       <origin xyz="0 0 0" rpy="${-M_PI/2} 0 ${-M_PI/2}" />
-      <parent link="${name}_rgb_frame" />
-      <child link="${name}_rgb_optical_frame" />
+      <parent link="camera_rgb_frame" />
+      <child link="camera_rgb_optical_frame" />
     </joint>
-    <link name="${name}_rgb_optical_frame">
+    <link name="camera_rgb_optical_frame">
       <inertial>
         <mass value="0.001" />
@@ -65,13 +39,22 @@
       </inertial>
     </link>
-  <!-- The fixed joints & links below are usually published by static_transformers launched by the OpenNi launch
-       files. However, for Gazebo simulation we need them, so we add them here.
-       (Hence, don't publish them additionally!) -->
-  <joint name="${name}_depth_joint" type="fixed">
-    <origin xyz="0.031 +0.0127 0.016" rpy="0 0 0" />
-    <parent link="${name}_link" />
-    <child link="${name}_depth_frame" />
+  <joint name="camera_joint" type="fixed">
+    <origin xyz="-0.031 ${-cam_py} -0.016" rpy="0 0 0"/>
+    <parent link="camera_rgb_frame"/>
+    <child link="camera_link"/>
   </joint>
-  <link name="${name}_depth_frame">
+  <link name="camera_link">
+    <visual>
+     <origin xyz="0 0 0" rpy="0 0 ${M_PI/2}"/>
+      <geometry>
+       <mesh filename="package://husky_fei_description/meshes/sensors/kinect.dae"/>
+      </geometry>
+    </visual>
+    <collision>
+      <origin xyz="0.0 0.0 0.0" rpy="0 0 0"/>
+      <geometry>
+	<box size="0.07271 0.27794 0.073"/>
+      </geometry>
+    </collision>
     <inertial>
       <mass value="0.001" />
@@ -82,10 +65,27 @@
     </inertial>
   </link>
-  <joint name="${name}_depth_optical_joint" type="fixed">
+  <!-- The fixed joints & links below are usually published by static_transformers launched by the OpenNi launch
+       files. However, for Gazebo simulation we need them, so we add them here.
+       (Hence, don't publish them additionally!) -->
+  <joint name="camera_depth_joint" type="fixed">
+    <origin xyz="0 ${2 * -cam_py} 0" rpy="0 0 0" />
+    <parent link="camera_rgb_frame" />
+    <child link="camera_depth_frame" />
+  </joint>
+  <link name="camera_depth_frame">
+    <inertial>
+      <mass value="0.001" />
+      <origin xyz="0 0 0" />
+      <inertia ixx="0.0001" ixy="0.0" ixz="0.0"
+               iyy="0.0001" iyz="0.0"
+               izz="0.0001" />
+    </inertial>
+  </link>
+  <joint name="camera_depth_optical_joint" type="fixed">
     <origin xyz="0 0 0" rpy="${-M_PI/2} 0 ${-M_PI/2}" />
-    <parent link="${name}_depth_frame" />
-    <child link="${name}_depth_optical_frame" />
+    <parent link="camera_depth_frame" />
+    <child link="camera_depth_optical_frame" />
   </joint>
-  <link name="${name}_depth_optical_frame">
+  <link name="camera_depth_optical_frame">
     <inertial>
       <mass value="0.001" />

File: husky_fei_description/urdf/sensors/microstrain_3dmgx2_imu.gazebo.xacro (robot description, xacro)
@@ -1,7 +1,7 @@
 <?xml version="1.0"?>
-<robot xmlns:xacro="http://ros.org/wiki/xacro">
-  <xacro:macro name="microstrain_3dmgx2_imu_gazebo_v0" params="name imu_topic update_rate stdev">
+<robot name="imusensor_gazebo" xmlns:xacro="http://ros.org/wiki/xacro">
+  <xacro:macro name="microstrain_3dmgx2_imu_gazebo" params="name imu_topic update_rate stdev">
     <gazebo>
-      <plugin name="imu_controller" filename="libgazebo_ros_imu.so">
+      <plugin name="gazebo_ros_${name}_controller" filename="libgazebo_ros_imu.so">
         <alwaysOn>true</alwaysOn>
         <updateRate>${update_rate}</updateRate>

File: husky_fei_description/urdf/sensors/microstrain_3dmgx2_imu.urdf.xacro (robot description, xacro)
@@ -3,10 +3,4 @@
   <xacro:include filename="$(find husky_fei_description)/urdf/sensors/microstrain_3dmgx2_imu.gazebo.xacro" />
   <xacro:macro name="sensor_imu" params="name parent colour imu_px imu_py imu_pz imu_or imu_op imu_oy imu_topic update_rate stdev">
-    <joint name="${name}_joint" type="fixed">
-      <axis xyz="0 1 0" />
-      <origin xyz="${imu_px} ${imu_py} ${imu_pz}" rpy="${imu_or} ${imu_op} ${imu_oy}"/>
-      <parent link="${parent}_link"/>
-      <child link="${name}_link"/>
-    </joint>
     <link name="${name}_link">
       <inertial>
@@ -31,6 +25,11 @@
 -->
     </link>
+    <joint name="${name}_joint" type="fixed">
+      <parent link="${parent}"/>
+      <child link="${name}_link"/>
+      <origin xyz="${imu_px} ${imu_py} ${imu_pz}" rpy="${imu_or} ${imu_op} ${imu_oy}"/>
+    </joint>
     <!-- gazebo extensions -->
-    <xacro:microstrain_3dmgx2_imu_gazebo_v0 name="${name}" imu_topic="${imu_topic}" update_rate="${update_rate}" stdev="${stdev}" />
+    <xacro:microstrain_3dmgx2_imu_gazebo_ name="${name}" imu_topic="${imu_topic}" update_rate="${update_rate}" stdev="${stdev}" />
   </xacro:macro>
 </robot>
