Commit message: Stereo camera appears to be properly configured now

File: husky_fei_description/urdf/husky_fei.urdf (robot description, URDF)
Before this commit: robot husky_fei, 24 links, 23 joints
Links:
- added link base_footprint_fei_stereo_rail_part, mass 0.1; collision box size=0.02 0.02 0.3; visual mesh filename=package://husky_fei_description/meshes/tslot_500x20x20.dae
- added link camera_depth_frame, mass 0.001
- added link camera_depth_optical_frame, mass 0.001
- added link camera_link, mass 0.001; collision box size=0.07271 0.27794 0.073; visual mesh filename=package://husky_fei_description/meshes/sensors/kinect.dae
- added link camera_rgb_frame, mass 0.001
- added link camera_rgb_optical_frame, mass 0.001
- link base_footprint_fei_gps_rail_part: geometry collision box size=0.02 0.02 0.4; visual mesh filename=package://husky_fei_description/meshes/tslot_200x20x20.dae
- link gps_link: geometry collision box size=0.096 0.096 0.096; visual mesh filename=package://husky_fei_description/meshes/sensors/GPSAntennaSc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
Joints:
- added joint base_footprint_fei_stereo_rail_joint: type fixed, parent base_footprint, child base_footprint_fei_stereo_rail_part, origin xyz=-0.24 0.0 0.63092492 rpy=1.57079632679 0.0 0.0
- added joint camera_depth_joint: type fixed, parent camera_link, child camera_depth_frame, origin xyz=0.031 +0.0127 0.016 rpy=0 0 0
- added joint camera_depth_optical_joint: type fixed, parent camera_depth_frame, child camera_depth_optical_frame, origin xyz=0 0 0 rpy=-1.57079632679 0 -1.57079632679
- added joint camera_joint: type fixed, parent base_link, child camera_link, origin xyz=-0.151 0.0 0.58092492 rpy=0.0 0.0 0.0
- added joint camera_rgb_joint: type fixed, parent camera_link, child camera_rgb_frame, origin xyz=0.031 -0.0127 0.016 rpy=0 0 0
- added joint camera_rgb_optical_joint: type fixed, parent camera_rgb_frame, child camera_rgb_optical_frame, origin xyz=0 0 0 rpy=-1.57079632679 0 -1.57079632679
- joint base_footprint_fei_gps_rail_joint: origin xyz=-0.15 0.18 0.58092492 rpy=1.57079632679 0.0 0.0 -> xyz=-0.15 0.18 0.49092492 rpy=0.0 0.0 0.0
- joint gps_joint: origin xyz=-0.151 0.182 0.61392492 rpy=0.0 0.0 3.14159265359 -> xyz=-0.151 0.18 0.48392492 rpy=0.0 0.0 3.14159265359
- joint left_camera_joint: origin xyz=0 0.031 0 rpy=0 0 0 -> xyz=0.025 0.031 0 rpy=0 0 0
- joint right_camera_joint: origin xyz=0 -0.031 0 rpy=0 0 0 -> xyz=0.025 -0.031 0 rpy=0 0 0
- joint stereo_camera_joint: origin xyz=-0.15 0.0 0.54092492 rpy=0.0 0.0 0.0 -> xyz=-0.24 0.0 0.75092492 rpy=0.0 0.0 0.0

File: husky_fei_description/urdf/husky_fei.urdf.xacro (robot description, xacro)
@@ -160,7 +160,7 @@
     <sensor_kinect name="camera" parent="base_link" cam_px="-0.12" cam_py="0.0" cam_pz="${0.207 + 0.245 + wheel_x_size/2 - base_z_origin_to_wheel_origin}" cam_or="0.0" cam_op="0.0" cam_oy="0.0" />
     <!-- FEI-modded vertical-stereo-camera rail -->
-    <husky_rail_mods parent="base_footprint" name="fei_stereo_rail" mesh="tslot_450x20x20"
-          colour="DarkGrey"
-          translateX="-0.24" translateY="0.0" translateZ="${0.216 + 0.245 + wheel_x_size/2 - base_z_origin_to_wheel_origin}"
+    <husky_rail_mods parent="base_footprint" name="fei_stereo_rail" mesh="tslot_500x20x20"
+          colour="DarkGrey"
+          translateX="-0.24" translateY="0.0" translateZ="${0.241 + 0.245 + wheel_x_size/2 - base_z_origin_to_wheel_origin}"
           rotateX="${M_PI/2.0}" rotateY="0.0" rotateZ="0.0" dimX="0.02" dimY="0.02" dimZ="0.3" />
     <gazebo reference="base_footprint_fei_stereo_rail_part">
@@ -168,6 +168,5 @@
     </gazebo>
     <!-- FEI-modded multicamera sensor -->
-    <sensor_multicamera name="stereo_camera" parent="base_link" baseline="0.062" colour="Red" cam_px="-0.24" cam_py="0.0" cam_pz="${0.311 + 0.245 + wheel_x_size/2 - base_z_origin_to_wheel_origin}" cam_or="0.0" cam_op="0.0" cam_oy="0.0" />
-<!--
+    <sensor_multicamera name="stereo_camera" parent="base_link" baseline="0.062" colour="Red" cam_px="-0.24" cam_py="0.0" cam_pz="${0.361 + 0.245 + wheel_x_size/2 - base_z_origin_to_wheel_origin}" cam_or="0.0" cam_op="0.0" cam_oy="0.0" />
     <gazebo reference="stereo_camera_link">
         <material>Gazebo/Red</material>
@@ -179,5 +178,4 @@
         <material>Gazebo/Black</material>
     </gazebo>
--->
     <!-- FEI-modded IMU sensor -->
     <!--<sensor_imu name="imu" parent="base" colour="Blue" imu_px="0.192" imu_py="0.0" imu_pz="${0.05 + wheel_x_size/2 - base_z_origin_to_wheel_origin}" imu_or="0.0" imu_op="${M_PI/2.0}" imu_oy="0.0" imu_topic="imu_data" update_rate="100.0" stdev="1.7e-2" /> -->

File: husky_fei_description/urdf/sensors/multicamera.gazebo.xacro (robot description, xacro)
@@ -6,5 +6,7 @@
         <update_rate>60.0</update_rate>
         <camera name="left">
-          <pose>0 ${baseline/2.0} 0 0 0 0</pose>
+<!-- x = 0.035 because the face of the red box is +0.05m/2 = 0.025m from origin +
+         0.01m for the black circle -->
+          <pose>0.035 ${baseline/2.0} 0 0 0 0</pose>
           <!-- <horizontal_fov>1.3962634</horizontal_fov> -->
           <horizontal_fov>${3.1415926535897931/2.0}</horizontal_fov>
@@ -25,5 +27,7 @@
         </camera>
         <camera name="right">
-          <pose>0 ${-baseline/2.0} 0 0 0 0</pose>
+<!-- x = 0.035 because the face of the red box is +0.05m/2 = 0.025m from origin +
+         0.01m for the black circle -->
+          <pose>0.035 ${-baseline/2.0} 0 0 0 0</pose>
           <!-- <horizontal_fov>1.3962634</horizontal_fov> -->
           <horizontal_fov>${3.1415926535897931/2.0}</horizontal_fov>

File: husky_fei_description/urdf/sensors/multicamera.urdf.xacro (robot description, xacro)
@@ -17,14 +17,14 @@
       </inertial>
       <visual>
-        <origin xyz="0 0 0" rpy="0 0 -1.57079632679" />
-<!--
+        <origin xyz="0 0 0" rpy="0 0 0" />
           <geometry>
             <box size="0.05 0.1 0.05" />
           </geometry>
           <material name="${colour}" />
--->
+<!--
 	<geometry>
           <mesh filename="package://husky_fei_description/meshes/sensors/PS3eye_stereo.dae" />
 	</geometry>
+-->
       </visual>
       <collision>
@@ -36,12 +36,11 @@
     </link>
     <joint name="left_camera_joint" type="fixed">
-      <origin xyz="0 ${baseline/2.0} 0" rpy="0 0 0" />
+      <origin xyz="0.025 ${baseline/2.0} 0" rpy="0 0 0" />
       <parent link="${name}_link" />
       <child link="left_camera_frame" />
     </joint>
     <link name="left_camera_frame">
-<!--
       <visual>
-        <origin xyz="0.025 0 0" rpy="0 1.57079632679 0" />
+        <origin xyz="0 0 0" rpy="0 1.57079632679 0" />
           <geometry>
             <cylinder radius="0.01" length="0.01" />
@@ -49,15 +48,13 @@
           <material name="Black" />
       </visual>
--->
     </link>
     <joint name="right_camera_joint" type="fixed">
-      <origin xyz="0 ${-baseline/2.0} 0" rpy="0 0 0" />
+      <origin xyz="0.025 ${-baseline/2.0} 0" rpy="0 0 0" />
       <parent link="${name}_link" />
       <child link="right_camera_frame" />
     </joint>
     <link name="right_camera_frame">
-<!--
       <visual>
-        <origin xyz="0.025 0 0" rpy="0 1.57079632679 0" />
+        <origin xyz="0 0 0" rpy="0 1.57079632679 0" />
           <geometry>
             <cylinder radius="0.01" length="0.01" />
@@ -65,5 +62,4 @@
           <material name="Black" />
       </visual>
--->
     </link>
   <!-- gazebo extension -->

Commit message: Point cloud registration appears to be fixed; laser scanner settings must be reviewed

File: husky_fei_description/urdf/husky_fei.urdf (robot description, URDF)
Before this commit: robot husky_fei, 30 links, 29 joints
Links:
- link base_footprint_fei_gps_rail_part: geometry collision box size=0.02 0.02 0.2; visual mesh filename=package://husky_fei_description/meshes/tslot_200x20x20.dae
- link base_footprint_fei_stereo_rail_part: geometry collision box size=0.02 0.02 0.5; visual mesh filename=package://husky_fei_description/meshes/tslot_500x20x20.dae
- link gps_link: geometry collision box size=0.096 0.096 0.084; visual mesh filename=package://husky_fei_description/meshes/sensors/GPSAntennaSc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
- link laser_link: geometry collision box size=0.122 0.104 0.175; visual mesh filename=package://husky_fei_description/meshes/sensors/LMS100.dae
- link left_camera_frame: mass None -> 0.001
- link right_camera_frame: mass None -> 0.001
- link stereo_camera_link: geometry collision box size=0.06 0.11 0.06; visual cylinder length=0.1 radius=0.025
Joints:
- joint base_footprint_fei_stereo_rail_joint: origin xyz=-0.24 0.0 0.63092492 rpy=1.57079632679 0.0 0.0 -> xyz=-0.24 0.0 0.63092492 rpy=0.0 0.0 0.0
- joint left_camera_joint: origin xyz=0.025 0.031 0 rpy=0 0 0 -> xyz=0.030 0.031 0 rpy=0 0 0
- joint right_camera_joint: origin xyz=0.025 -0.031 0 rpy=0 0 0 -> xyz=0.030 -0.031 0 rpy=0 0 0

File: husky_fei_description/urdf/husky_fei.urdf.xacro (robot description, xacro)
@@ -157,6 +157,6 @@
         <material>Gazebo/Grey</material>
     </gazebo>
-    <!-- FEI-modded 3D sensor -->
-    <sensor_kinect name="camera" parent="base_link" cam_px="-0.12" cam_py="0.0" cam_pz="${0.207 + 0.245 + wheel_x_size/2 - base_z_origin_to_wheel_origin}" cam_or="0.0" cam_op="0.0" cam_oy="0.0" />
+    <!-- FEI-modded 3D sensor cam_pz: 0.151 works well too, but must change rail -->
+    <sensor_kinect name="camera" parent="base_link" cam_px="-0.151" cam_py="0.0" cam_pz="${0.191 + 0.245 + wheel_x_size/2 - base_z_origin_to_wheel_origin}" cam_or="0.0" cam_op="0.0" cam_oy="0.0" />
     <!-- FEI-modded vertical-stereo-camera rail -->
     <husky_rail_mods parent="base_footprint" name="fei_stereo_rail" mesh="tslot_500x20x20"

File: husky_fei_description/urdf/sensors/3dsensor_gazebo.urdf.xacro (robot description, xacro)
@@ -3,10 +3,11 @@
   <!-- Microsoft Kinect / ASUS Xtion PRO Live for simulation -->
   <xacro:macro name="husky_fei_sim_3dsensor" params="name">
-    <gazebo reference="${name}_link">
-      <sensor type="depth" name="${name}">
+    <!-- <gazebo reference="${name}_link">  -->
+    <gazebo reference="${name}_depth_frame">
+      <sensor type="depth" name="${name}_frame_sensor">
         <always_on>true</always_on>
         <update_rate>30.0</update_rate>
         <camera>
-          <horizontal_fov>${60.0*M_PI/180.0}</horizontal_fov>
+          <horizontal_fov>${57.0*M_PI/180.0}</horizontal_fov>
           <image>
             <format>R8G8B8</format>
@@ -15,6 +16,6 @@
           </image>
           <clip>
-            <near>0.01</near>
-            <far>8.0</far>
+            <near>0.1</near>
+            <far>100.0</far>
           </clip>
         </camera>
@@ -28,16 +29,11 @@
           <depthImageCameraInfoTopicName>depth/camera_info</depthImageCameraInfoTopicName>
           <frameName>${name}_depth_optical_frame</frameName>
-          <baseline>0.1</baseline>
-          <distortion_k1>0.0</distortion_k1>
-          <distortion_k2>0.0</distortion_k2>
-          <distortion_k3>0.0</distortion_k3>
-          <distortion_t1>0.0</distortion_t1>
-          <distortion_t2>0.0</distortion_t2>
           <pointCloudCutoff>0.4</pointCloudCutoff>
-          <CxPrime>0</CxPrime>
-          <Cx>0</Cx>
-          <Cy>0</Cy>
-          <focalLength>0</focalLength>
-          <hackBaseline>0</hackBaseline>
+          <distortion_k1>0.00000001</distortion_k1>
+          <distortion_k2>0.00000001</distortion_k2>
+          <distortion_k3>0.00000001</distortion_k3>
+          <distortion_t1>0.00000001</distortion_t1>
+          <distortion_t2>0.00000001</distortion_t2>
+          <!-- <baseline>0.2</baseline> -->
         </plugin>
       </sensor>

File: husky_fei_description/urdf/sensors/kinect.urdf.xacro (robot description, xacro)
@@ -12,5 +12,5 @@
   <xacro:macro name="sensor_kinect" params="name parent cam_px cam_py cam_pz cam_or cam_op cam_oy">
     <joint name="${name}_joint" type="fixed">
-      <origin xyz="${cam_px - 0.031} ${cam_py} ${cam_pz - 0.016}" rpy="${cam_or} ${cam_op} ${cam_oy}"/>
+      <origin xyz="${cam_px} ${cam_py} ${cam_pz - 0.015}" rpy="${cam_or} ${cam_op} ${cam_oy}"/>
       <parent link="${parent}"/>
       <child link="${name}_link" />
@@ -19,5 +19,5 @@
       <inertial>
         <mass value="0.001" />
-        <origin xyz="0 0 0" />
+        <origin xyz="0 0 0.0" />
         <inertia ixx="0.0001" ixy="0.0" ixz="0.0"
                  iyy="0.0001" iyz="0.0"
@@ -25,5 +25,5 @@
       </inertial>
       <visual>
-        <origin xyz="0 0 0" rpy="0 0 ${M_PI/2}"/>
+        <origin xyz="0 0 0.015" rpy="0 0 ${M_PI/2}"/>
           <geometry>
             <mesh filename="package://husky_fei_description/meshes/sensors/kinect.dae"/>
@@ -38,5 +38,5 @@
     </link>
     <joint name="${name}_rgb_joint" type="fixed">
-      <origin xyz="0.031 -0.0127 0.016" rpy="0 0 0"/>
+      <origin xyz="0.031 -0.0127 0.031" rpy="0 0 0"/>
       <parent link="${name}_link"/>
       <child link="${name}_rgb_frame"/>
@@ -68,5 +68,5 @@
        (Hence, don't publish them additionally!) -->
   <joint name="${name}_depth_joint" type="fixed">
-    <origin xyz="0.031 +0.0127 0.016" rpy="0 0 0" />
+    <origin xyz="0.031 +0.0127 0.031" rpy="0 0 0" />
     <parent link="${name}_link" />
     <child link="${name}_depth_frame" />
