Commit message: Frames now have a prefix parameter passed to main xacro file to ensure heterogeneous tf trees without the use of (deprecated) tf_prefix

File: husky_fei_description/urdf/husky_fei.urdf (robot description, URDF)
Before this commit: robot husky_fei, 30 links, 29 joints
Links:
- removed link back_left_wheel
- removed link back_right_wheel
- removed link baro_link
- removed link base_footprint
- removed link base_footprint_fei_cam_rail_part
- removed link base_footprint_fei_gps_rail_part
- removed link base_footprint_fei_hb_rail_part
- removed link base_footprint_fei_hf_rail_part
- removed link base_footprint_fei_lms100_l_rail_part
- removed link base_footprint_fei_lms100_r_rail_part
- removed link base_footprint_fei_stereo_rail_part
- removed link base_footprint_front_bumper_part
- removed link base_footprint_lms100_support_part
- removed link base_footprint_rear_bumper_part
- removed link base_footprint_top_plate_part
- removed link base_footprint_user_rail_part
- removed link base_link
- removed link camera_depth_frame
- removed link camera_depth_optical_frame
- removed link camera_link
- removed link camera_rgb_frame
- removed link camera_rgb_optical_frame
- removed link front_left_wheel
- removed link front_right_wheel
- removed link gps_link
- removed link imu_link
- removed link laser_link
- removed link left_camera_frame
- removed link right_camera_frame
- removed link stereo_camera_link
- added link husky_back_left_wheel, mass 2.63657; collision cylinder length=0.1143 radius=0.17775; visual mesh filename=package://husky_fei_description/meshes/wheel.stl
- added link husky_back_right_wheel, mass 2.63657; collision cylinder length=0.1143 radius=0.17775; visual mesh filename=package://husky_fei_description/meshes/wheel.stl
- added link husky_baro_link, mass 0.10; visual box size=0.01 0.02 0.02
- added link husky_base_footprint; visual box size=0.001 0.001 0.001
- added link husky_base_footprint_fei_cam_rail_part, mass 0.1; collision box size=0.02 0.02 0.3; visual mesh filename=package://husky_fei_description/meshes/tslot_300x20x20.dae
- added link husky_base_footprint_fei_gps_rail_part, mass 0.1; collision box size=0.02 0.02 0.2; visual mesh filename=package://husky_fei_description/meshes/tslot_200x20x20.dae
- added link husky_base_footprint_fei_hb_rail_part, mass 0.1; collision box size=0.001 0.001 0.001; visual mesh filename=package://husky_fei_description/meshes/tslot_400x20x20.dae
- added link husky_base_footprint_fei_hf_rail_part, mass 0.1; collision box size=0.001 0.001 0.001; visual mesh filename=package://husky_fei_description/meshes/tslot_400x20x20.dae
- added link husky_base_footprint_fei_lms100_l_rail_part, mass 0.1; collision box size=0.02 0.02 0.1; visual mesh filename=package://husky_fei_description/meshes/tslot_100x20x20.dae
- added link husky_base_footprint_fei_lms100_r_rail_part, mass 0.1; collision box size=0.02 0.02 0.1; visual mesh filename=package://husky_fei_description/meshes/tslot_100x20x20.dae
- added link husky_base_footprint_fei_stereo_rail_part, mass 0.1; collision box size=0.02 0.02 0.5; visual mesh filename=package://husky_fei_description/meshes/tslot_500x20x20.dae
- added link husky_base_footprint_front_bumper_part, mass 0.1; collision box size=0.001 0.001 0.001; visual mesh filename=package://husky_fei_description/meshes/bumper.stl
- added link husky_base_footprint_lms100_support_part, mass 0.1; collision box size=0.02 0.02 0.1; visual mesh filename=package://husky_fei_description/meshes/sensors/LMS100_suppo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
- added link husky_base_footprint_rear_bumper_part, mass 0.1; collision box size=0.001 0.001 0.001; visual mesh filename=package://husky_fei_description/meshes/bumper.stl
- added link husky_base_footprint_top_plate_part, mass 0.1; collision box size=0.001 0.001 0.001; visual mesh filename=package://husky_fei_description/meshes/top_plate.stl
- added link husky_base_footprint_user_rail_part, mass 0.1; collision box size=0.001 0.001 0.001; visual mesh filename=package://husky_fei_description/meshes/user_rail.stl
- added link husky_base_link, mass 33.45489; collision box size=1.0074 0.5709 0.2675; visual mesh filename=package://husky_fei_description/meshes/base_link.stl
- added link husky_camera_depth_frame, mass 0.001
- added link husky_camera_depth_optical_frame, mass 0.001
- added link husky_camera_link, mass 0.001; collision box size=0.07271 0.27794 0.073; visual mesh filename=package://husky_fei_description/meshes/sensors/kinect.dae
- added link husky_camera_rgb_frame, mass 0.001
- added link husky_camera_rgb_optical_frame, mass 0.001
- added link husky_front_left_wheel, mass 2.63657; collision cylinder length=0.1143 radius=0.17775; visual mesh filename=package://husky_fei_description/meshes/wheel.stl
- added link husky_front_right_wheel, mass 2.63657; collision cylinder length=0.1143 radius=0.17775; visual mesh filename=package://husky_fei_description/meshes/wheel.stl
- added link husky_gps_link, mass 0.10; collision box size=0.096 0.096 0.084; visual mesh filename=package://husky_fei_description/meshes/sensors/GPSAntennaSc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
- added link husky_imu_link, mass 0.01; visual box size=0.025 0.025 0.01
- added link husky_laser_link, mass 1.1; collision box size=0.122 0.104 0.175; visual mesh filename=package://husky_fei_description/meshes/sensors/LMS100.dae
- added link husky_left_camera_frame, mass 0.001; visual cylinder length=0.01 radius=0.01
- added link husky_right_camera_frame, mass 0.001; visual cylinder length=0.01 radius=0.01
- added link husky_stereo_camera_link, mass 0.01; collision box size=0.06 0.11 0.06; visual cylinder length=0.1 radius=0.025
Joints:
- removed joint baro_joint
- removed joint base_footprint_fei_cam_rail_joint
- removed joint base_footprint_fei_gps_rail_joint
- removed joint base_footprint_fei_hb_rail_joint
- removed joint base_footprint_fei_hf_rail_joint
- removed joint base_footprint_fei_lms100_l_rail_joint
- removed joint base_footprint_fei_lms100_r_rail_joint
- removed joint base_footprint_fei_stereo_rail_joint
- removed joint base_footprint_front_bumper_joint
- removed joint base_footprint_joint
- removed joint base_footprint_lms100_support_joint
- removed joint base_footprint_rear_bumper_joint
- removed joint base_footprint_top_plate_joint
- removed joint base_footprint_user_rail_joint
- removed joint camera_depth_joint
- removed joint camera_depth_optical_joint
- removed joint camera_joint
- removed joint camera_rgb_joint
- removed joint camera_rgb_optical_joint
- removed joint gps_joint
- removed joint imu_joint
- removed joint joint_back_left_wheel
- removed joint joint_back_right_wheel
- removed joint joint_front_left_wheel
- removed joint joint_front_right_wheel
- removed joint laser_joint
- removed joint left_camera_joint
- removed joint right_camera_joint
- removed joint stereo_camera_joint
- added joint husky_baro_joint: type fixed, parent husky_base_link, child husky_baro_link, origin xyz=0.192 -0.05 0.19492492 rpy=0.0 0.0 0.0
- added joint husky_base_footprint_fei_cam_rail_joint: type fixed, parent husky_base_footprint, child husky_base_footprint_fei_cam_rail_part, origin xyz=-0.15 0.0 0.54092492 rpy=0.0 0.0 0.0
- added joint husky_base_footprint_fei_gps_rail_joint: type fixed, parent husky_base_footprint, child husky_base_footprint_fei_gps_rail_part, origin xyz=-0.15 0.18 0.49092492 rpy=0.0 0.0 0.0
- added joint husky_base_footprint_fei_hb_rail_joint: type fixed, parent husky_base_footprint, child husky_base_footprint_fei_hb_rail_part, origin xyz=-0.15 0.0 0.38092492 rpy=0.0 0.0 0.0
- added joint husky_base_footprint_fei_hf_rail_joint: type fixed, parent husky_base_footprint, child husky_base_footprint_fei_hf_rail_part, origin xyz=0.21 0.0 0.38092492 rpy=0.0 0.0 0.0
- added joint husky_base_footprint_fei_lms100_l_rail_joint: type fixed, parent husky_base_footprint, child husky_base_footprint_fei_lms100_l_rail_part, origin xyz=0.242 -0.035 0.42092492 rpy=0.0 0.0 0.0
- added joint husky_base_footprint_fei_lms100_r_rail_joint: type fixed, parent husky_base_footprint, child husky_base_footprint_fei_lms100_r_rail_part, origin xyz=0.242 0.035 0.42092492 rpy=0.0 0.0 0.0
- added joint husky_base_footprint_fei_stereo_rail_joint: type fixed, parent husky_base_footprint, child husky_base_footprint_fei_stereo_rail_part, origin xyz=-0.24 0.0 0.63092492 rpy=0.0 0.0 0.0
- added joint husky_base_footprint_front_bumper_joint: type fixed, parent husky_base_footprint, child husky_base_footprint_front_bumper_part, origin xyz=0.49 0.0 0.23592492 rpy=0.0 0.0 0.0
- added joint husky_base_footprint_joint: type fixed, parent husky_base_footprint, child husky_base_link, origin xyz=0 0 0.14492492 rpy=0 0 0
- added joint husky_base_footprint_lms100_support_joint: type fixed, parent husky_base_footprint, child husky_base_footprint_lms100_support_part, origin xyz=0.314 0.0 0.47992492 rpy=0.0 0.0 0.0
- added joint husky_base_footprint_rear_bumper_joint: type fixed, parent husky_base_footprint, child husky_base_footprint_rear_bumper_part, origin xyz=-0.48 0.0 0.23592492 rpy=0.0 0.0 3.14
- added joint husky_base_footprint_top_plate_joint: type fixed, parent husky_base_footprint, child husky_base_footprint_top_plate_part, origin xyz=0.0 0.0 0.14492492 rpy=0.0 0.0 0.0
- added joint husky_base_footprint_user_rail_joint: type fixed, parent husky_base_footprint, child husky_base_footprint_user_rail_part, origin xyz=0.272 0.0 0.38992492 rpy=0.0 0.0 0.0
- added joint husky_camera_depth_joint: type fixed, parent husky_camera_link, child husky_camera_depth_frame, origin xyz=0.031 +0.0127 0.031 rpy=0 0 0
- added joint husky_camera_depth_optical_joint: type fixed, parent husky_camera_depth_frame, child husky_camera_depth_optical_frame, origin xyz=0 0 0 rpy=-1.57079632679 0 -1.57079632679
- added joint husky_camera_joint: type fixed, parent husky_base_link, child husky_camera_link, origin xyz=-0.151 0.0 0.56592492 rpy=0.0 0.0 0.0
- added joint husky_camera_rgb_joint: type fixed, parent husky_camera_link, child husky_camera_rgb_frame, origin xyz=0.031 -0.0127 0.031 rpy=0 0 0
- added joint husky_camera_rgb_optical_joint: type fixed, parent husky_camera_rgb_frame, child husky_camera_rgb_optical_frame, origin xyz=0 0 0 rpy=-1.57079632679 0 -1.57079632679
- added joint husky_gps_joint: type fixed, parent husky_base_link, child husky_gps_link, origin xyz=-0.151 0.18 0.48392492 rpy=0.0 0.0 3.14159265359
- added joint husky_imu_joint: type fixed, parent husky_base_link, child husky_imu_link, origin xyz=0.192 0.0 0.19492492 rpy=0.0 -1.57079632679 0.0
- added joint husky_joint_back_left_wheel: type continuous, parent husky_base_link, child husky_back_left_wheel, origin xyz=-0.25600006 0.285475 0.03282508 rpy=0 0 0, axis 0 1 0, limit effort=100 velocity=100
- added joint husky_joint_back_right_wheel: type continuous, parent husky_base_link, child husky_back_right_wheel, origin xyz=-0.25600006 -0.285475 0.03282508 rpy=0 0 0, axis 0 1 0, limit effort=100 velocity=100
- added joint husky_joint_front_left_wheel: type continuous, parent husky_base_link, child husky_front_left_wheel, origin xyz=0.25600006 0.285475 0.03282508 rpy=0 0 0, axis 0 1 0, limit effort=100 velocity=100
- added joint husky_joint_front_right_wheel: type continuous, parent husky_base_link, child husky_front_right_wheel, origin xyz=0.25600006 -0.285475 0.03282508 rpy=0 0 0, axis 0 1 0, limit effort=100 velocity=100
- added joint husky_laser_joint: type fixed, parent husky_base_link, child husky_laser_link, origin xyz=0.314 0.0 0.28492492 rpy=0.0 0.0 0
- added joint husky_left_camera_joint: type fixed, parent husky_stereo_camera_link, child husky_left_camera_frame, origin xyz=0.030 0.031 0 rpy=0 0 0
- added joint husky_right_camera_joint: type fixed, parent husky_stereo_camera_link, child husky_right_camera_frame, origin xyz=0.030 -0.031 0 rpy=0 0 0
- added joint husky_stereo_camera_joint: type fixed, parent husky_base_link, child husky_stereo_camera_link, origin xyz=-0.24 0.0 0.75092492 rpy=0.0 0.0 0.0
