Commit message: Frames now have a prefix parameter passed to main xacro file to ensure heterogeneous tf trees without the use of (deprecated) tf_prefix

File: husky_fei_description/urdf/sensors/kingfisher_imu_gazebo.urdf.xacro (robot description, xacro)
@@ -6,9 +6,9 @@
 	<always_on>true</always_on>
         <update_rate>100.0</update_rate>
-        <bodyName>${name}_link</bodyName>
+        <bodyName>$(arg prefix)_${name}_link</bodyName>
         <topicName>${name}_data</topicName>
         <serviceName>${name}_service</serviceName>
-        <rpyOffsets>0 0 0</rpyOffsets> <!-- deprecated -->
-        <gaussianNoise>0</gaussianNoise> <!-- deprecated -->
+        <rpyOffset>0 0 0</rpyOffset>
+        <gaussianNoise>0</gaussianNoise>
         <accelDrift>0.5 0.5 0.5</accelDrift>
         <accelGaussianNoise>0.35 0.35 0.3</accelGaussianNoise>

File: husky_fei_description/urdf/sensors/multicamera.gazebo.xacro (robot description, xacro)
@@ -2,5 +2,5 @@
 <robot name="multicamera_gazebo" xmlns:xacro="http://ros.org/wiki/xacro">
   <xacro:macro name="husky_fei_sim_multicamera" params="name baseline">
-    <gazebo reference="${name}_link">
+    <gazebo reference="$(arg prefix)_${name}_link">
       <sensor type="multicamera" name="${name}">
         <update_rate>60.0</update_rate>
@@ -49,5 +49,5 @@
           <imageTopicName>image_raw</imageTopicName>
           <cameraInfoTopicName>${name}_info</cameraInfoTopicName>
-          <frameName>left_camera_frame</frameName>
+          <frameName>$(arg prefix)_left_camera_frame</frameName>
           <hackBaseline>${baseline}</hackBaseline>
           <distortionK1>0.0</distortionK1>

File: husky_fei_description/urdf/sensors/sick_lms100_gpu_laser.gazebo.xacro (robot description, xacro)
@@ -2,5 +2,5 @@
 <robot xmlns:xacro="http://ros.org/wiki/xacro">
   <xacro:macro name="sick_lms100_gpu_laser_gazebo" params="name">
-    <gazebo reference="${name}_link">
+    <gazebo reference="$(arg prefix)_${name}_link">
       <sensor type="gpu_ray" name="${name}_lms100_gpu_sensor">
         <always_on>true</always_on>

File: husky_fei_description/urdf/sensors/sick_lms100_laser.gazebo.xacro (robot description, xacro)
@@ -2,5 +2,5 @@
 <robot xmlns:xacro="http://ros.org/wiki/xacro">
   <xacro:macro name="sick_lms100_laser_gazebo" params="name">
-    <gazebo reference="${name}_link">
+    <gazebo reference="$(arg prefix)_${name}_link">
       <sensor type="ray" name="${name}_lms100_sensor">
         <always_on>true</always_on>

File: husky_fei_description/urdf/sensors/sick_lms100_laser.urdf.xacro (robot description, xacro)
@@ -3,11 +3,11 @@
   <xacro:include filename="$(find husky_fei_description)/urdf/sensors/sick_lms100_laser.gazebo.xacro" />
   <xacro:macro name="sick_lms100_laser" params="name parent laser_px laser_py laser_pz laser_or laser_op laser_oy">
-    <joint name="${name}_joint" type="fixed">
+    <joint name="$(arg prefix)_${name}_joint" type="fixed">
       <!-- <axis xyz="0 1 0" /> -->
       <origin xyz="${laser_px} ${laser_py} ${laser_pz}" rpy="${laser_or} ${laser_op} ${laser_oy}"/>
       <parent link="${parent}"/>
-      <child link="${name}_link"/>
+      <child link="$(arg prefix)_${name}_link"/>
     </joint>
-    <link name="${name}_link" type="laser">
+    <link name="$(arg prefix)_${name}_link" type="laser">
       <inertial>
         <mass value="1.1" />
