Commit message: multicamera properly configured with TF and offsets all matching

File: husky_fei_description/urdf/sensors/multicamera.gazebo.xacro (robot description, xacro)
@@ -6,7 +6,5 @@
         <update_rate>60.0</update_rate>
         <camera name="left">
-<!-- x = 0.035 because the face of the red box is +0.05m/2 = 0.025m from origin +
-         0.01m for the black circle -->
-          <pose>0.035 ${baseline/2.0} 0 0 0 0</pose>
+          <pose>0.030 ${baseline/2.0} 0 0 0 0</pose>
           <!-- <horizontal_fov>1.3962634</horizontal_fov> -->
           <horizontal_fov>${3.1415926535897931/2.0}</horizontal_fov>
@@ -27,7 +25,5 @@
         </camera>
         <camera name="right">
-<!-- x = 0.035 because the face of the red box is +0.05m/2 = 0.025m from origin +
-         0.01m for the black circle -->
-          <pose>0.035 ${-baseline/2.0} 0 0 0 0</pose>
+          <pose>0.030 ${-baseline/2.0} 0 0 0 0</pose>
           <!-- <horizontal_fov>1.3962634</horizontal_fov> -->
           <horizontal_fov>${3.1415926535897931/2.0}</horizontal_fov>
@@ -53,5 +49,5 @@
           <imageTopicName>image_raw</imageTopicName>
           <cameraInfoTopicName>${name}_info</cameraInfoTopicName>
-          <frameName>${name}_left_camera_optical_frame</frameName>
+          <frameName>left_camera_frame</frameName>
           <hackBaseline>${baseline}</hackBaseline>
           <distortionK1>0.0</distortionK1>

File: husky_fei_description/urdf/sensors/multicamera.urdf.xacro (robot description, xacro)
@@ -17,7 +17,8 @@
       </inertial>
       <visual>
-        <origin xyz="0 0 0" rpy="0 0 0" />
+        <origin xyz="0 0 0" rpy="1.57079632679 0 0" />
           <geometry>
-            <box size="0.05 0.1 0.05" />
+            <!-- <box size="0.05 0.1 0.05" /> -->
+            <cylinder radius="0.025" length="0.1" />
           </geometry>
           <material name="${colour}" />
@@ -31,16 +32,23 @@
         <origin xyz="0.0 0.0 0.0" rpy="0 0 0" />
         <geometry>
-          <box size="0.05 0.1 0.05" />
+          <box size="0.06 0.11 0.06" />
         </geometry>
       </collision>
     </link>
     <joint name="left_camera_joint" type="fixed">
-      <origin xyz="0.025 ${baseline/2.0} 0" rpy="0 0 0" />
+      <origin xyz="0.030 ${baseline/2.0} 0" rpy="0 0 0" />
       <parent link="${name}_link" />
       <child link="left_camera_frame" />
     </joint>
     <link name="left_camera_frame">
+      <inertial>
+        <mass value="0.001" />
+        <origin xyz="0 0 0" />
+        <inertia ixx="0.0001" ixy="0.0" ixz="0.0"
+                 iyy="0.0001" iyz="0.0"
+                 izz="0.0001" />
+      </inertial>
       <visual>
-        <origin xyz="0 0 0" rpy="0 1.57079632679 0" />
+        <origin xyz="-0.005 0 0" rpy="0 1.57079632679 0" />
           <geometry>
             <cylinder radius="0.01" length="0.01" />
@@ -50,11 +58,18 @@
     </link>
     <joint name="right_camera_joint" type="fixed">
-      <origin xyz="0.025 ${-baseline/2.0} 0" rpy="0 0 0" />
+      <origin xyz="0.030 ${-baseline/2.0} 0" rpy="0 0 0" />
       <parent link="${name}_link" />
       <child link="right_camera_frame" />
     </joint>
     <link name="right_camera_frame">
+      <inertial>
+        <mass value="0.001" />
+        <origin xyz="0 0 0" />
+        <inertia ixx="0.0001" ixy="0.0" ixz="0.0"
+                 iyy="0.0001" iyz="0.0"
+                 izz="0.0001" />
+      </inertial>
       <visual>
-        <origin xyz="0 0 0" rpy="0 1.57079632679 0" />
+        <origin xyz="-0.005 0 0" rpy="0 1.57079632679 0" />
           <geometry>
             <cylinder radius="0.01" length="0.01" />
