Commit message: Corrected collision settings for laser

File: husky_fei_description/urdf/sensors/sick_lms100_laser.urdf.xacro (robot description, xacro)
@@ -18,5 +18,5 @@
         <origin xyz="0 0 0.05" rpy="0 0 0"/>
         <geometry>
-          <box size="0.120 0.102 0.165"/>
+          <box size="0.122 0.104 0.175"/>
         </geometry>
       </collision>

Commit message: Correction for upside-down laser -- should check if Gazebo sim is OK

File: husky_fei_description/urdf/sensors/sick_lms100_laser.urdf.xacro (robot description, xacro)
@@ -12,9 +12,9 @@
       <inertial>
         <mass value="1.1" />
-        <origin xyz="0 0 0.05" rpy="0 0 0" />
+        <origin xyz="0 0 -0.05" rpy="3.1415926535897931 0 0" />
         <inertia ixx="0.0001" ixy="0" ixz="0" iyy="0.000001" iyz="0" izz="0.0001" />
       </inertial>
       <collision>
-        <origin xyz="0 0 0.05" rpy="0 0 0"/>
+        <origin xyz="0 0 -0.05" rpy="3.1415926535897931 0 0"/>
         <geometry>
           <box size="0.122 0.104 0.175"/>
@@ -22,5 +22,5 @@
       </collision>
       <visual>
-        <origin xyz="0 0 0.05" rpy="0 0 0"/>
+        <origin xyz="0 0 -0.05" rpy="3.1415926535897931 0 0"/>
         <geometry>
           <mesh filename="package://husky_fei_description/meshes/sensors/LMS100.dae"/>
